File: a500_pwr.sch (KiCad schematic (older format))
At the start: 20 parts, among them J1 PJ-102A, J2 APWR_big, J3 APWR_small, SW1 RMS1R102M7QES, U1 LMZM23600SILR, U2 RPM5.0-6.0

Commit message: Waiver
Parts:
- C1: Herstellernr. C3216X5R1H106K160AB -> (none)
- C2: Herstellernr. (none) -> C2012X7R2A104K125AA
- C3, C4: Herstellernr. (none) -> CGA5L1X7R1V106K160AC
- C6: Herstellernr. (none) -> C3216X5R1H106K160AB
- D1: DK_Detail_Page (none) -> /product-detail/de/diodes-incorporated/B360A-13-F/B360A-FDI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; Description (none) -> DIODE SCHOTTKY 60V 3A SMA; Herstellernr. (none) -> B360A-13-F; Manufacturer (none) -> Diodes Incorporated
- J3: Description (none) -> 3 pin header 2.54mm
- L1: DK_Detail_Page (none) -> product-detail/de/würth-elektronik/742792510/732-1640-1-ND/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; Description (none) -> FERRITE BEAD 70 OHM 1812 1LN; Digi-Key_PN (none) -> 732-1640-1-ND; Herstellernr. (none) -> 742792510
- L2: DK_Detail_Page (none) -> /product-detail/de/würth-elektronik/7427932/732-2394-1-ND/2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; Description (none) -> FERRITE BEAD 98 OHM 2SMD 1LN; Digi-Key_PN (none) -> 732-2394-1-ND; Herstellernr. (none) -> 7427932
- R3, R4: Description (none) -> optional 5V adjust
- SW1: DK_Detail_Page (none) -> /products/de?keywords=RMS1R102M7QES; Description (none) -> SWITCH ROCKER SPDT 3A 120V; Digi-Key_PN (none) -> 450-2074-ND; Herstellernr. (none) -> RMS1R102M7QES
- U1: value LMZM23600SILR -> LMZM23600SILT; DK_Detail_Page (none) -> /product-detail/de/texas-instruments/LMZM23600SILT/296-4945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; Description (none) -> DC DC CONVERTER 2.5-15V; Digi-Key_PN (none) -> 296-49457-1-ND; Herstellernr. (none) -> LMZM23600SILT; Manufacturer (none) -> Texas Instruments
- U2: DK_Detail_Page (none) -> /product-detail/de/recom-power/RPM5-0-6-0/945-3256-1-ND/964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; Description (none) -> 6A DC/DC-CONVERTER 'INNOLINE' SM; Digi-Key_PN (none) -> 945-3256-1-ND
Changed lines of the file:
@@
 P 7750 5200
 F 0 "U1" H 7750 5725 50  0000 C CNN
-F 1 "LMZM23600SILR" H 7750 5634 50  0000 C CNN
+F 1 "LMZM23600SILT" H 7750 5634 50  0000 C CNN
 F 2 "a500_pwr:SIL0010A" H 8100 5150 50  0001 C CNN
 F 3 "http://www.ti.com/general/docs/suppproductinfo.tsp?distId=26&gotoUrl=http%3A%2F%2Fwww.ti.com%2Flit%2Fds%2Fsymlink%2Flmzm23600.pdf" H 8100 5150 50  0001 C CNN
+F 4 "/product-detail/de/texas-instruments/LMZM23600SILT/296-49457-1-ND/9371296" H 7750 5200 50  0001 C CNN "DK_Detail_Page"
+F 5 "DC DC CONVERTER 2.5-15V" H 7750 5200 50  0001 C CNN "Description"
+F 6 "296-49457-1-ND" H 7750 5200 50  0001 C CNN "Digi-Key_PN"
+F 7 "LMZM23600SILT" H 7750 5200 50  0001 C CNN "Herstellernr."
+F 8 "Texas Instruments" H 7750 5200 50  0001 C CNN "Manufacturer"
 	1    7750 5200
 	1    0    0    -1
@@
 F 1 "100n 50V" H 6492 5155 50  0000 L CNN
 F 2 "Capacitors_SMD:C_0805_HandSoldering" H 6400 5200 50  0001 C CNN
-F 3 "C2012X7R2A104K125AA" H 6400 5200 50  0001 C CNN
+F 3 "" H 6400 5200 50  0001 C CNN
+F 4 "C2012X7R2A104K125AA" H 6400 5200 50  0001 C CNN "Herstellernr."
 	1    6400 5200
 	1    0    0    -1
@@
 F 1 "10u 25V" H 5992 5155 50  0000 L CNN
 F 2 "Capacitors_SMD:C_1206_HandSoldering" H 5900 5200 50  0001 C CNN
-F 3 "https://www.mouser.de/datasheet/2/400/lcc_commercial_general_en-837201.pdf" H 5900 5200 50  0001 C CNN
-F 4 "C3216X5R1H106K160AB" H 5900 5200 50  0001 C CNN "Herstellernr."
+F 3 "" H 5900 5200 50  0001 C CNN
+F 4 "" H 5900 5200 50  0001 C CNN "Herstellernr."
 	1    5900 5200
 	1    0    0    -1
@@
 F 1 "10u" H 9492 5255 50  0000 L CNN
 F 2 "Capacitors_SMD:C_1206_HandSoldering" H 9400 5300 50  0001 C CNN
-F 3 "CGA5L1X7R1V106K160AC" H 9400 5300 50  0001 C CNN
+F 3 "" H 9400 5300 50  0001 C CNN
+F 4 "CGA5L1X7R1V106K160AC" H 9400 5300 50  0001 C CNN "Herstellernr."
 	1    9400 5300
 	1    0    0    -1
@@
 F 1 "10u" H 9792 5255 50  0000 L CNN
 F 2 "Capacitors_SMD:C_1206_HandSoldering" H 9700 5300 50  0001 C CNN
-F 3 "CGA5L1X7R1V106K160AC" H 9700 5300 50  0001 C CNN
+F 3 "" H 9700 5300 50  0001 C CNN
+F 4 "CGA5L1X7R1V106K160AC" H 9700 5300 50  0001 C CNN "Herstellernr."
 	1    9700 5300
 	1    0    0    -1
@@
 F 1 "700mV" V 10095 5368 50  0000 L CNN
 F 2 "Diodes_SMD:D_SMA_Handsoldering" V 10050 5300 50  0001 C CNN
-F 3 "B360A-13-F" V 10050 5300 50  0001 C CNN
+F 3 "" V 10050 5300 50  0001 C CNN
+F 4 "/product-detail/de/diodes-incorporated/B360A-13-F/B360A-FDICT-ND/724980" H 10050 5300 50  0001 C CNN "DK_Detail_Page"
+F 5 "DIODE SCHOTTKY 60V 3A SMA" H 10050 5300 50  0001 C CNN "Description"
+F 6 "B360A-13-F" H 10050 5300 50  0001 C CNN "Herstellernr."
+F 7 "Diodes Incorporated" H 10050 5300 50  0001 C CNN "Manufacturer"
 	1    10050 5300
 	0    1    1    0
@@
 F 1 "APWR_big" H 8480 1901 50  0000 L CNN
 F 2 "a500_pwr:APWR_big" H 8400 2000 50  0001 C CNN
-F 3 "~" H 8400 2000 50  0001 C CNN
+F 3 "" H 8400 2000 50  0001 C CNN
 	1    8400 2000
 	1    0    0    -1
@@
 F 1 "APWR_small" H 8480 2601 50  0000 L CNN
 F 2 "a500_pwr:APWR_small" H 8400 2650 50  0001 C CNN
-F 3 "~" H 8400 2650 50  0001 C CNN
+F 3 "" H 8400 2650 50  0001 C CNN
 F 4 "Connectors, Headers" H 8400 2650 50  0001 C CNN "Category"
+F 5 "3 pin header 2.54mm" H 8400 2650 50  0001 C CNN "Description"
 	1    8400 2650
 	1    0    0    -1
@@
 F 2 "a500_pwr:RPM5.0-6.0" H 2000 4000 50  0001 C CNN
 F 3 "https://www.mouser.de/datasheet/2/468/RPM-6.0-1398219.pdf" V 2350 4500 50  0001 C CNN
+F 4 "/product-detail/de/recom-power/RPM5-0-6-0/945-3256-1-ND/9644705" H 2500 4750 50  0001 C CNN "DK_Detail_Page"
+F 5 "6A DC/DC-CONVERTER 'INNOLINE' SM" H 2500 4750 50  0001 C CNN "Description"
+F 6 "945-3256-1-ND" H 2500 4750 50  0001 C CNN "Digi-Key_PN"
 	1    2500 4750
 	1    0    0    -1
@@
 F 2 "a500_pwr:RPM5.0-6.0" H 1750 5300 50  0001 C CNN
 F 3 "https://www.mouser.de/datasheet/2/468/RPM-6.0-1398219.pdf" V 2100 5800 50  0001 C CNN
+F 4 "/product-detail/de/recom-power/RPM5-0-6-0/945-3256-1-ND/9644705" H 2250 6050 50  0001 C CNN "DK_Detail_Page"
+F 5 "6A DC/DC-CONVERTER 'INNOLINE' SM" H 2250 6050 50  0001 C CNN "Description"
+F 6 "945-3256-1-ND" H 2250 6050 50  0001 C CNN "Digi-Key_PN"
 	2    2250 6050
 	-1   0    0    1
@@
 F 3 "https://www.mouser.de/datasheet/2/445/742792510-1720733.pdf" H 1400 4250 50  0001 C CNN
 F 4 "Würth" H 1400 4250 50  0001 C CNN "Manufacturer"
+F 5 "product-detail/de/würth-elektronik/742792510/732-1640-1-ND/1639584" H 1400 4250 50  0001 C CNN "DK_Detail_Page"
+F 6 "FERRITE BEAD 70 OHM 1812 1LN" H 1400 4250 50  0001 C CNN "Description"
+F 7 "732-1640-1-ND" H 1400 4250 50  0001 C CNN "Digi-Key_PN"
+F 8 "742792510" H 1400 4250 50  0001 C CNN "Herstellernr."
 	1    1400 4250
 	0    1    1    0
@@
 F 3 "https://www.mouser.de/datasheet/2/445/7427932-1720978.pdf" H 3450 4250 50  0001 C CNN
 F 4 "Würth" H 3450 4250 50  0001 C CNN "Manufacturer"
+F 5 "/product-detail/de/würth-elektronik/7427932/732-2394-1-ND/2268596" H 3450 4250 50  0001 C CNN "DK_Detail_Page"
+F 6 "FERRITE BEAD 98 OHM 2SMD 1LN" H 3450 4250 50  0001 C CNN "Description"
+F 7 "732-2394-1-ND" H 3450 4250 50  0001 C CNN "Digi-Key_PN"
+F 8 "7427932" H 3450 4250 50  0001 C CNN "Herstellernr."
 	1    3450 4250
 	0    1    1    0
@@
 F 1 "10u 25V" H 1242 4405 50  0000 L CNN
 F 2 "Capacitors_SMD:C_1206_HandSoldering" H 1150 4450 50  0001 C CNN
-F 3 "C3216X5R1H106K160AB" H 1150 4450 50  0001 C CNN
+F 3 "" H 1150 4450 50  0001 C CNN
 	1    1150 4450
 	1    0    0    -1
@@
 F 1 "22u" H 3842 4455 50  0000 L CNN
 F 2 "Capacitors_SMD:C_1206_HandSoldering" H 3750 4500 50  0001 C CNN
-F 3 "C3216X5R1H106K160AB" H 3750 4500 50  0001 C CNN
+F 3 "" H 3750 4500 50  0001 C CNN
+F 4 "C3216X5R1H106K160AB" H 3750 4500 50  0001 C CNN "Herstellernr."
 	1    3750 4500
 	1    0    0    -1
@@
 F 2 "Capacitors_SMD:C_0603_HandSoldering" H 3300 4550 50  0001 C CNN
 F 3 "" H 3300 4550 50  0001 C CNN
+F 4 "optional 5V adjust" H 3300 4550 50  0001 C CNN "Description"
 	1    3300 4550
 	-1   0    0    1
@@
 F 2 "Capacitors_SMD:C_0603_HandSoldering" H 3300 4750 50  0001 C CNN
 F 3 "" H 3300 4750 50  0001 C CNN
+F 4 "optional 5V adjust" H 3300 4750 50  0001 C CNN "Description"
 	1    3300 4750
 	-1   0    0    1
@@
 F 1 "330u" H 5115 3105 50  0000 L CNN
 F 2 "Capacitors_THT:CP_Radial_D8.0mm_P3.50mm" H 5038 3000 50  0001 C CNN
-F 3 "~" H 5000 3150 50  0001 C CNN
+F 3 "" H 5000 3150 50  0001 C CNN
 	1    5000 3150
 	1    0    0    -1
@@
 F 3 "https://www.mouser.de/datasheet/2/418/NG_CD_2267087_A_2267087_c.dwg-680380.pdf" H 5000 2100 50  0001 C CNN
 F 4 "" H 5000 2100 50  0001 C CNN "Feld4"
+F 5 "/products/de?keywords=RMS1R102M7QES" H 5000 2100 50  0001 C CNN "DK_Detail_Page"
+F 6 "SWITCH ROCKER SPDT 3A 120V" H 5000 2100 50  0001 C CNN "Description"
+F 7 "450-2074-ND" H 5000 2100 50  0001 C CNN "Digi-Key_PN"
+F 8 "RMS1R102M7QES" H 5000 2100 50  0001 C CNN "Herstellernr."
 	1    5000 2100
 	1    0    0    -1

Commit message: adjust for different Barrel connector and note about R3/R4
Other:
- note added: "R3/R4 are optional\nto adjust the output voltage"
Changed lines of the file:
@@
 	7000 5150 7000 5750
 NoConn ~ 5000 2200
+Text Notes 3450 5350 0    50   ~ 0
+R3/R4 are optional\nto adjust the output voltage
 $EndSCHEMATC
