File: a500_pwr.sch (KiCad schematic (older format))
At the start: 20 parts, among them J1 PJ-102A, J2 APWR_big, J3 APWR_small, SW1 RMS1R102M7QES, U1 LMZM23600SILT, U2 RPM5.0-6.0

Commit message: fix 22µF Mouser part number
Parts:
- C6: Herstellernr. C3216X5R1H106K160AB -> C3216X5R1V226M160AC
Changed lines of the file:
@@
 F 2 "Capacitors_SMD:C_1206_HandSoldering" H 3750 4500 50  0001 C CNN
 F 3 "" H 3750 4500 50  0001 C CNN
-F 4 "C3216X5R1H106K160AB" H 3750 4500 50  0001 C CNN "Herstellernr."
+F 4 "C3216X5R1V226M160AC" H 3750 4500 50  0001 C CNN "Herstellernr."
 	1    3750 4500
 	1    0    0    -1
