File: a500_pwr.kicad_pcb (KiCad board)
At the start: 2 copper layers, 28.8 x 43.8 mm, 20 parts, among them J1 PJ-102A, J2 APWR_big, J3 APWR_small, SW1 RMS1R102M7QES, U1 LMZM23600SILR, U2 RPM5.0-6.0

Commit message: for real now with new gerbers
Parts:
- U1: value LMZM23600SILR -> LMZM23600SILT
Connections:
- U1 pad 5: (no net) -> Net-(U1-Pad5)

Commit message: thickend all 12V and 5V traces
Routing:
- net GND: track 78.1 -> 8.24 mm, vias 21 -> 26
- net +12V: track 50.9 -> 55.9 mm, vias 2 -> 4
- added copper zone on F.Cu, net +5V
- added copper zone on F.Cu, net /SW12V
- added copper zone on F.Cu, net Net-(L1-Pad1)
- added copper zone on F.Cu, net Net-(L2-Pad2)
Other:
- board text added: "Rev. 4"
- board text removed: "Rev. 3"
